Commit message: modify gazebo and xacro

File: example/flying_gazebo_stereo_cam/model/flying_stereo_cam.xacro (robot description, xacro)
@@ -43,5 +43,5 @@
 	<origin xyz="0 0 0" rpy="0 0 0"/>
 	<geometry>
-	  <box size="${cameraSize*2} ${cameraSize} ${cameraSize}"/>
+	  <box size="${cameraSize*2*0} ${cameraSize*0} ${cameraSize*0}"/>
 	</geometry>
       </collision>
